File: schema/MotoGuzziJiffy.sch (KiCad schematic (older format))
At the start: 6 parts

Commit message: Weet niet, zag dat de fets er niet inzaten
Parts:
- added Q?: IRLML0030TRPBF, SOT23, symbol IRF7309IPBF
- added Q?: IRLML2244TRPBF, TO220, symbol IRF9540N
- added R? (x2): R, ~, symbol R
Connections:
- wire segments 8 -> 15
Changed lines of the file:
@@
 Sheet 1 1
 Title ""
-Date "16 feb 2015"
+Date "17 feb 2015"
 Rev ""
 Comp ""
@@
 	1    0    0    -1
 $EndComp
+$Comp
+L IRF7309IPBF Q?
+U 1 1 54E3C3E1
+P 4700 5200
+F 0 "Q?" H 4700 5052 40  0000 R CNN
+F 1 "IRLML0030TRPBF" H 4700 5349 40  0000 R CNN
+F 2 "SOT23" H 4521 5301 29  0000 C CNN
+F 3 "" H 4700 5200 60  0000 C CNN
+	1    4700 5200
+	1    0    0    -1
+$EndComp
+$Comp
+L IRF9540N Q?
+U 1 1 54E3C4CD
+P 5100 4250
+F 0 "Q?" H 5100 4102 40  0000 R CNN
+F 1 "IRLML2244TRPBF" H 5100 4399 40  0000 R CNN
+F 2 "TO220" H 4881 4351 29  0000 C CNN
+F 3 "" H 5100 4250 60  0000 C CNN
+	1    5100 4250
+	1    0    0    -1
+$EndComp
+$Comp
+L R R?
+U 1 1 54E3C5A0
+P 4800 3750
+F 0 "R?" V 4880 3750 40  0000 C CNN
+F 1 "R" V 4807 3751 40  0000 C CNN
+F 2 "~" V 4730 3750 30  0000 C CNN
+F 3 "~" H 4800 3750 30  0000 C CNN
+	1    4800 3750
+	1    0    0    -1
+$EndComp
+$Comp
+L R R?
+U 1 1 54E3C649
+P 4800 4750
+F 0 "R?" V 4880 4750 40  0000 C CNN
+F 1 "R" V 4807 4751 40  0000 C CNN
+F 2 "~" V 4730 4750 30  0000 C CNN
+F 3 "~" H 4800 4750 30  0000 C CNN
+	1    4800 4750
+	1    0    0    -1
+$EndComp
+Wire Wire Line
+	4800 4000 4800 4500
+Wire Wire Line
+	4900 4300 4800 4300
+Connection ~ 4800 4300
+Wire Wire Line
+	2850 -1000 3300 -1000
+Wire Wire Line
+	2650 2800 2300 2800
+Wire Wire Line
+	2300 2800 2300 5250
+Wire Wire Line
+	2300 5250 4500 5250
+Wire Wire Line
+	4500 5250 4500 5300
 $EndSCHEMATC

Commit message: Wat voortgang
Parts:
- removed Q?: IRLML2244TRPBF, TO220, symbol IRF9540N
- added P1: CONN_3X2, symbol CONN_3X2
- added Q?: IRLML2244TRPBF, SOT-23, symbol IRLML2244TRPBF
- R5, R6: renamed from R?; value R -> 1k
- gave numbers to parts that had none: 1
Connections:
- net labels added: Lamp
- wire segments 15 -> 20
Changed lines of the file:
@@
 LIBS:contrib
 LIBS:valves
+LIBS:kiCadCarl
 LIBS:MotoGuzziJiffy-cache
 EELAYER 27 0
@@
 Sheet 1 1
 Title ""
-Date "17 feb 2015"
+Date "24 feb 2015"
 Rev ""
 Comp ""
@@
 $EndComp
 $Comp
-L IRF7309IPBF Q?
+L IRF7309IPBF Q1
 U 1 1 54E3C3E1
 P 4700 5200
-F 0 "Q?" H 4700 5052 40  0000 R CNN
+F 0 "Q1" H 4700 5052 40  0000 R CNN
 F 1 "IRLML0030TRPBF" H 4700 5349 40  0000 R CNN
 F 2 "SOT23" H 4521 5301 29  0000 C CNN
@@
 $EndComp
 $Comp
-L IRF9540N Q?
-U 1 1 54E3C4CD
+L R R5
+U 1 1 54E3C5A0
+P 4800 3750
+F 0 "R5" V 4880 3750 40  0000 C CNN
+F 1 "1k" V 4807 3751 40  0000 C CNN
+F 2 "~" V 4730 3750 30  0000 C CNN
+F 3 "~" H 4800 3750 30  0000 C CNN
+	1    4800 3750
+	1    0    0    -1
+$EndComp
+$Comp
+L R R6
+U 1 1 54E3C649
+P 4800 4750
+F 0 "R6" V 4880 4750 40  0000 C CNN
+F 1 "1k" V 4807 4751 40  0000 C CNN
+F 2 "~" V 4730 4750 30  0000 C CNN
+F 3 "~" H 4800 4750 30  0000 C CNN
+	1    4800 4750
+	1    0    0    -1
+$EndComp
+Wire Wire Line
+	4800 4000 4800 4500
+Wire Wire Line
+	4900 4300 4800 4300
+Connection ~ 4800 4300
+Wire Wire Line
+	2850 -1000 3300 -1000
+Wire Wire Line
+	2650 2800 2300 2800
+Wire Wire Line
+	2300 2800 2300 5250
+Wire Wire Line
+	2300 5250 4500 5250
+Wire Wire Line
+	4500 5250 4500 5300
+$Comp
+L CONN_3X2 P1
+U 1 1 54ECEB1F
+P 3050 3650
+F 0 "P1" H 3050 3900 50  0000 C CNN
+F 1 "CONN_3X2" V 3050 3700 40  0000 C CNN
+F 2 "" H 3050 3650 60  0000 C CNN
+F 3 "" H 3050 3650 60  0000 C CNN
+	1    3050 3650
+	1    0    0    -1
+$EndComp
+$Comp
+L IRLML2244TRPBF Q?
+U 1 1 54ED03E4
 P 5100 4250
 F 0 "Q?" H 5100 4102 40  0000 R CNN
 F 1 "IRLML2244TRPBF" H 5100 4399 40  0000 R CNN
-F 2 "TO220" H 4881 4351 29  0000 C CNN
-F 3 "" H 5100 4250 60  0000 C CNN
+F 2 "SOT-23" H 4881 4351 29  0000 C CNN
+F 3 "~" H 5100 4250 60  0000 C CNN
 	1    5100 4250
 	1    0    0    -1
 $EndComp
-$Comp
-L R R?
-U 1 1 54E3C5A0
-P 4800 3750
-F 0 "R?" V 4880 3750 40  0000 C CNN
-F 1 "R" V 4807 3751 40  0000 C CNN
-F 2 "~" V 4730 3750 30  0000 C CNN
-F 3 "~" H 4800 3750 30  0000 C CNN
-	1    4800 3750
-	1    0    0    -1
-$EndComp
-$Comp
-L R R?
-U 1 1 54E3C649
-P 4800 4750
-F 0 "R?" V 4880 4750 40  0000 C CNN
-F 1 "R" V 4807 4751 40  0000 C CNN
-F 2 "~" V 4730 4750 30  0000 C CNN
-F 3 "~" H 4800 4750 30  0000 C CNN
-	1    4800 4750
-	1    0    0    -1
-$EndComp
-Wire Wire Line
-	4800 4000 4800 4500
-Wire Wire Line
-	4900 4300 4800 4300
-Connection ~ 4800 4300
-Wire Wire Line
-	2850 -1000 3300 -1000
-Wire Wire Line
-	2650 2800 2300 2800
-Wire Wire Line
-	2300 2800 2300 5250
-Wire Wire Line
-	2300 5250 4500 5250
-Wire Wire Line
-	4500 5250 4500 5300
+Wire Wire Line
+	5200 4450 5500 4450
+Wire Wire Line
+	5500 4450 5500 3450
+Wire Wire Line
+	4800 3500 4800 3450
+Wire Wire Line
+	4800 3450 5750 3450
+Wire Wire Line
+	5200 4050 5750 4050
+Text Label 5600 3400 0    60   ~ 0
++12V
+Text Label 5600 4000 0    60   ~ 0
+Lamp
 $EndSCHEMATC

Commit message: p fet nu met drain naar beneden
Parts:
- added U?: 78L05, symbol 78L05
Connections:
- net labels added: LAMP
- net labels removed: Lamp
- wire segments 20 -> 24
Changed lines of the file:
@@
 Sheet 1 1
 Title ""
-Date "24 feb 2015"
+Date "25 feb 2015"
 Rev ""
 Comp ""
@@
 $EndComp
 Wire Wire Line
-	5200 4450 5500 4450
-Wire Wire Line
-	5500 4450 5500 3450
-Wire Wire Line
 	4800 3500 4800 3450
 Wire Wire Line
 	4800 3450 5750 3450
-Wire Wire Line
-	5200 4050 5750 4050
 Text Label 5600 3400 0    60   ~ 0
 +12V
-Text Label 5600 4000 0    60   ~ 0
-Lamp
+Wire Wire Line
+	5200 4050 5200 3450
+Connection ~ 5200 3450
+Wire Wire Line
+	5200 4450 5750 4450
+Text Label 5500 4450 0    60   ~ 0
+LAMP
+$Comp
+L GND #PWR?
+U 1 1 54EE5528
+P 4800 5550
+F 0 "#PWR?" H 4800 5550 30  0001 C CNN
+F 1 "GND" H 4800 5480 30  0001 C CNN
+F 2 "" H 4800 5550 60  0000 C CNN
+F 3 "" H 4800 5550 60  0000 C CNN
+	1    4800 5550
+	1    0    0    -1
+$EndComp
+Wire Wire Line
+	4800 5400 4800 5550
+$Comp
+L GND #PWR?
+U 1 1 54EE554F
+P 5350 3200
+F 0 "#PWR?" H 5350 3200 30  0001 C CNN
+F 1 "GND" H 5350 3130 30  0001 C CNN
+F 2 "" H 5350 3200 60  0000 C CNN
+F 3 "" H 5350 3200 60  0000 C CNN
+	1    5350 3200
+	1    0    0    -1
+$EndComp
+Wire Wire Line
+	5350 3100 5350 3200
+$Comp
+L 78L05 U?
+U 1 1 54EE5591
+P 4100 1900
+F 0 "U?" H 4250 1704 60  0000 C CNN
+F 1 "78L05" H 4100 2100 60  0000 C CNN
+F 2 "" H 4100 1900 60  0000 C CNN
+F 3 "" H 4100 1900 60  0000 C CNN
+	1    4100 1900
+	1    0    0    -1
+$EndComp
+$Comp
+L GND #PWR?
+U 1 1 54EE55A0
+P 4100 2300
+F 0 "#PWR?" H 4100 2300 30  0001 C CNN
+F 1 "GND" H 4100 2230 30  0001 C CNN
+F 2 "" H 4100 2300 60  0000 C CNN
+F 3 "" H 4100 2300 60  0000 C CNN
+	1    4100 2300
+	1    0    0    -1
+$EndComp
+Wire Wire Line
+	4100 2150 4100 2300
+Wire Wire Line
+	4500 1850 5350 1850
+Wire Wire Line
+	5350 1850 5350 2600
 $EndSCHEMATC

Commit message: ICSP header toegevoegd
Parts:
- P1: label (none) -> ICSP header
Connections:
- wire segments 24 -> 41
Other:
- moved on the sheet: IC?, P1, Q1A, R5, R6
Changed lines of the file:
@@
 Sheet 1 1
 Title ""
-Date "25 feb 2015"
+Date "6 mar 2015"
 Rev ""
 Comp ""
@@
 L ATTINY85-P IC?
 U 1 1 54B2F7E3
-P 4000 2850
-F 0 "IC?" H 2950 3250 60  0000 C CNN
-F 1 "ATTINY85-P" H 4850 2450 60  0000 C CNN
-F 2 "DIP8" H 2950 2450 60  0001 C CNN
-F 3 "" H 4000 2850 60  0000 C CNN
-	1    4000 2850
+P 4500 2850
+F 0 "IC?" H 3450 3250 60  0000 C CNN
+F 1 "ATTINY85-P" H 5350 2450 60  0000 C CNN
+F 2 "DIP8" H 3450 2450 60  0001 C CNN
+F 3 "" H 4500 2850 60  0000 C CNN
+	1    4500 2850
 	1    0    0    -1
 $EndComp
@@
 $EndComp
 Wire Wire Line
-	2550 2600 2650 2600
-Wire Wire Line
-	2550 2700 2650 2700
-Wire Wire Line
 	1800 2600 2050 2600
 Connection ~ 1800 2600
@@
 L IRF7309IPBF Q1
 U 1 1 54E3C3E1
-P 4700 5200
-F 0 "Q1" H 4700 5052 40  0000 R CNN
-F 1 "IRLML0030TRPBF" H 4700 5349 40  0000 R CNN
-F 2 "SOT23" H 4521 5301 29  0000 C CNN
-F 3 "" H 4700 5200 60  0000 C CNN
-	1    4700 5200
+P 4700 5650
+F 0 "Q1" H 4700 5502 40  0000 R CNN
+F 1 "IRLML0030TRPBF" H 4700 5799 40  0000 R CNN
+F 2 "SOT23" H 4521 5751 29  0000 C CNN
+F 3 "" H 4700 5650 60  0000 C CNN
+	1    4700 5650
 	1    0    0    -1
 $EndComp
@@
 L R R5
 U 1 1 54E3C5A0
-P 4800 3750
-F 0 "R5" V 4880 3750 40  0000 C CNN
-F 1 "1k" V 4807 3751 40  0000 C CNN
-F 2 "~" V 4730 3750 30  0000 C CNN
-F 3 "~" H 4800 3750 30  0000 C CNN
-	1    4800 3750
+P 4800 4200
+F 0 "R5" V 4880 4200 40  0000 C CNN
+F 1 "1k" V 4807 4201 40  0000 C CNN
+F 2 "~" V 4730 4200 30  0000 C CNN
+F 3 "~" H 4800 4200 30  0000 C CNN
+	1    4800 4200
 	1    0    0    -1
 $EndComp
@@
 L R R6
 U 1 1 54E3C649
-P 4800 4750
-F 0 "R6" V 4880 4750 40  0000 C CNN
-F 1 "1k" V 4807 4751 40  0000 C CNN
-F 2 "~" V 4730 4750 30  0000 C CNN
-F 3 "~" H 4800 4750 30  0000 C CNN
-	1    4800 4750
-	1    0    0    -1
-$EndComp
-Wire Wire Line
-	4800 4000 4800 4500
-Wire Wire Line
-	4900 4300 4800 4300
-Connection ~ 4800 4300
+P 4800 5200
+F 0 "R6" V 4880 5200 40  0000 C CNN
+F 1 "1k" V 4807 5201 40  0000 C CNN
+F 2 "~" V 4730 5200 30  0000 C CNN
+F 3 "~" H 4800 5200 30  0000 C CNN
+	1    4800 5200
+	1    0    0    -1
+$EndComp
+Wire Wire Line
+	4800 4450 4800 4950
+Connection ~ 4800 4750
 Wire Wire Line
 	2850 -1000 3300 -1000
-Wire Wire Line
-	2650 2800 2300 2800
-Wire Wire Line
-	2300 2800 2300 5250
-Wire Wire Line
-	2300 5250 4500 5250
 Wire Wire Line
 	4500 5250 4500 5300
@@
 L CONN_3X2 P1
 U 1 1 54ECEB1F
-P 3050 3650
-F 0 "P1" H 3050 3900 50  0000 C CNN
-F 1 "CONN_3X2" V 3050 3700 40  0000 C CNN
-F 2 "" H 3050 3650 60  0000 C CNN
-F 3 "" H 3050 3650 60  0000 C CNN
-	1    3050 3650
+P 3750 3650
+F 0 "P1" H 3750 3900 50  0000 C CNN
+F 1 "CONN_3X2" V 3750 3700 40  0000 C CNN
+F 2 "" H 3750 3650 60  0000 C CNN
+F 3 "" H 3750 3650 60  0000 C CNN
+F 4 "ICSP header" H 3750 3450 60  0000 C CNN "label"
+	1    3750 3650
 	1    0    0    -1
 $EndComp
@@
 L IRLML2244TRPBF Q?
 U 1 1 54ED03E4
-P 5100 4250
-F 0 "Q?" H 5100 4102 40  0000 R CNN
-F 1 "IRLML2244TRPBF" H 5100 4399 40  0000 R CNN
-F 2 "SOT-23" H 4881 4351 29  0000 C CNN
-F 3 "~" H 5100 4250 60  0000 C CNN
-	1    5100 4250
-	1    0    0    -1
-$EndComp
-Wire Wire Line
-	4800 3500 4800 3450
-Wire Wire Line
-	4800 3450 5750 3450
-Text Label 5600 3400 0    60   ~ 0
+P 5100 4700
+F 0 "Q?" H 5100 4552 40  0000 R CNN
+F 1 "IRLML2244TRPBF" H 5100 4849 40  0000 R CNN
+F 2 "SOT-23" H 4881 4801 29  0000 C CNN
+F 3 "~" H 5100 4700 60  0000 C CNN
+	1    5100 4700
+	1    0    0    -1
+$EndComp
+Wire Wire Line
+	4800 3950 4800 3900
+Wire Wire Line
+	4800 3900 5750 3900
+Text Label 5600 3850 0    60   ~ 0
 +12V
 Wire Wire Line
-	5200 4050 5200 3450
-Connection ~ 5200 3450
-Wire Wire Line
-	5200 4450 5750 4450
-Text Label 5500 4450 0    60   ~ 0
+	5200 4500 5200 3900
+Connection ~ 5200 3900
+Wire Wire Line
+	5200 4900 5750 4900
+Text Label 5500 4900 0    60   ~ 0
 LAMP
 $Comp
 L GND #PWR?
 U 1 1 54EE5528
-P 4800 5550
-F 0 "#PWR?" H 4800 5550 30  0001 C CNN
-F 1 "GND" H 4800 5480 30  0001 C CNN
-F 2 "" H 4800 5550 60  0000 C CNN
-F 3 "" H 4800 5550 60  0000 C CNN
-	1    4800 5550
-	1    0    0    -1
-$EndComp
-Wire Wire Line
-	4800 5400 4800 5550
+P 4800 6000
+F 0 "#PWR?" H 4800 6000 30  0001 C CNN
+F 1 "GND" H 4800 5930 30  0001 C CNN
+F 2 "" H 4800 6000 60  0000 C CNN
+F 3 "" H 4800 6000 60  0000 C CNN
+	1    4800 6000
+	1    0    0    -1
+$EndComp
+Wire Wire Line
+	4800 5850 4800 6000
 $Comp
 L GND #PWR?
 U 1 1 54EE554F
-P 5350 3200
-F 0 "#PWR?" H 5350 3200 30  0001 C CNN
-F 1 "GND" H 5350 3130 30  0001 C CNN
-F 2 "" H 5350 3200 60  0000 C CNN
-F 3 "" H 5350 3200 60  0000 C CNN
-	1    5350 3200
+P 5350 3650
+F 0 "#PWR?" H 5350 3650 30  0001 C CNN
+F 1 "GND" H 5350 3580 30  0001 C CNN
+F 2 "" H 5350 3650 60  0000 C CNN
+F 3 "" H 5350 3650 60  0000 C CNN
+	1    5350 3650
 	1    0    0    -1
 $EndComp
@@
 Wire Wire Line
 	5350 1850 5350 2600
+Wire Wire Line
+	2550 2600 3150 2600
+Wire Wire Line
+	2550 2700 3150 2700
+Wire Wire Line
+	2650 2700 2650 3500
+Wire Wire Line
+	2650 3500 3350 3500
+Connection ~ 2650 2700
+Wire Wire Line
+	4300 3600 4150 3600
+Wire Wire Line
+	6400 3500 6400 2600
+Wire Wire Line
+	6400 2600 5850 2600
+Wire Wire Line
+	3150 3100 2900 3100
+Wire Wire Line
+	2900 3100 2900 3700
+Wire Wire Line
+	2900 3700 3350 3700
+$Comp
+L GND #PWR?
+U 1 1 54F9D216
+P 4300 4000
+F 0 "#PWR?" H 4300 4000 30  0001 C CNN
+F 1 "GND" H 4300 3930 30  0001 C CNN
+F 2 "" H 4300 4000 60  0000 C CNN
+F 3 "" H 4300 4000 60  0000 C CNN
+	1    4300 4000
+	1    0    0    -1
+$EndComp
+Wire Wire Line
+	4150 3700 4300 3700
+Wire Wire Line
+	4300 3700 4300 4000
+Wire Wire Line
+	4150 3500 6400 3500
+Wire Wire Line
+	4300 3300 4300 3600
+Wire Wire Line
+	2750 3300 4300 3300
+Wire Wire Line
+	2750 3300 2750 2600
+Connection ~ 2750 2600
+Wire Wire Line
+	3150 2800 2950 2800
+Wire Wire Line
+	2950 2800 2950 3600
+Wire Wire Line
+	2950 3600 3350 3600
+Wire Wire Line
+	3150 2900 3050 2900
+Wire Wire Line
+	3050 2900 3050 5700
+Wire Wire Line
+	3050 5700 4500 5700
+Wire Wire Line
+	4800 4750 4900 4750
 $EndSCHEMATC

Commit message: Voedingslijntjes
Parts:
- added C1: 100 uF, ~, symbol C
- added R7: 1k, ~, symbol R
- R5, R6: value 1k -> 10k
Connections:
- wire segments 41 -> 45
Changed lines of the file:
@@
 	1    0    0    -1
 $EndComp
-Wire Wire Line
-	1800 1900 1800 3500
-Wire Wire Line
-	2000 1900 2000 3500
 $Comp
 L R R4
@@
 	0    1    1    0
 $EndComp
-Wire Wire Line
-	1800 2600 2050 2600
-Connection ~ 1800 2600
-Wire Wire Line
-	2000 2700 2050 2700
-Connection ~ 2000 2700
 $Comp
 L GND #PWR?
@@
 	1    0    0    -1
 $EndComp
-Wire Wire Line
-	1900 4500 1900 4650
-Wire Wire Line
-	1250 1400 2000 1400
 $Comp
 L +12V #PWR?
@@
 P 4800 4200
 F 0 "R5" V 4880 4200 40  0000 C CNN
-F 1 "1k" V 4807 4201 40  0000 C CNN
+F 1 "10k" V 4807 4201 40  0000 C CNN
 F 2 "~" V 4730 4200 30  0000 C CNN
 F 3 "~" H 4800 4200 30  0000 C CNN
@@
 P 4800 5200
 F 0 "R6" V 4880 5200 40  0000 C CNN
-F 1 "1k" V 4807 5201 40  0000 C CNN
+F 1 "10k" V 4807 5201 40  0000 C CNN
 F 2 "~" V 4730 5200 30  0000 C CNN
 F 3 "~" H 4800 5200 30  0000 C CNN
@@
 	1    0    0    -1
 $EndComp
-Wire Wire Line
-	4800 4450 4800 4950
-Connection ~ 4800 4750
-Wire Wire Line
-	2850 -1000 3300 -1000
-Wire Wire Line
-	4500 5250 4500 5300
 $Comp
 L CONN_3X2 P1
@@
 	1    0    0    -1
 $EndComp
-Wire Wire Line
-	4800 3950 4800 3900
-Wire Wire Line
-	4800 3900 5750 3900
 Text Label 5600 3850 0    60   ~ 0
 +12V
-Wire Wire Line
-	5200 4500 5200 3900
-Connection ~ 5200 3900
-Wire Wire Line
-	5200 4900 5750 4900
 Text Label 5500 4900 0    60   ~ 0
 LAMP
@@
 	1    0    0    -1
 $EndComp
-Wire Wire Line
-	4800 5850 4800 6000
 $Comp
 L GND #PWR?
 U 1 1 54EE554F
-P 5350 3650
-F 0 "#PWR?" H 5350 3650 30  0001 C CNN
-F 1 "GND" H 5350 3580 30  0001 C CNN
-F 2 "" H 5350 3650 60  0000 C CNN
-F 3 "" H 5350 3650 60  0000 C CNN
-	1    5350 3650
-	1    0    0    -1
-$EndComp
-Wire Wire Line
-	5350 3100 5350 3200
+P 5850 3200
+F 0 "#PWR?" H 5850 3200 30  0001 C CNN
+F 1 "GND" H 5850 3130 30  0001 C CNN
+F 2 "" H 5850 3200 60  0000 C CNN
+F 3 "" H 5850 3200 60  0000 C CNN
+	1    5850 3200
+	1    0    0    -1
+$EndComp
 $Comp
 L 78L05 U?
@@
 L GND #PWR?
 U 1 1 54EE55A0
-P 4100 2300
-F 0 "#PWR?" H 4100 2300 30  0001 C CNN
-F 1 "GND" H 4100 2230 30  0001 C CNN
-F 2 "" H 4100 2300 60  0000 C CNN
-F 3 "" H 4100 2300 60  0000 C CNN
-	1    4100 2300
-	1    0    0    -1
-$EndComp
-Wire Wire Line
-	4100 2150 4100 2300
-Wire Wire Line
-	4500 1850 5350 1850
-Wire Wire Line
-	5350 1850 5350 2600
-Wire Wire Line
-	2550 2600 3150 2600
-Wire Wire Line
-	2550 2700 3150 2700
-Wire Wire Line
-	2650 2700 2650 3500
-Wire Wire Line
-	2650 3500 3350 3500
-Connection ~ 2650 2700
-Wire Wire Line
-	4300 3600 4150 3600
-Wire Wire Line
-	6400 3500 6400 2600
-Wire Wire Line
-	6400 2600 5850 2600
-Wire Wire Line
-	3150 3100 2900 3100
-Wire Wire Line
-	2900 3100 2900 3700
-Wire Wire Line
-	2900 3700 3350 3700
+P 4100 2350
+F 0 "#PWR?" H 4100 2350 30  0001 C CNN
+F 1 "GND" H 4100 2280 30  0001 C CNN
+F 2 "" H 4100 2350 60  0000 C CNN
+F 3 "" H 4100 2350 60  0000 C CNN
+	1    4100 2350
+	1    0    0    -1
+$EndComp
 $Comp
 L GND #PWR?
@@
 $EndComp
 Wire Wire Line
+	1800 1900 1800 3500
+Wire Wire Line
+	2000 1900 2000 3500
+Wire Wire Line
+	1800 2600 2050 2600
+Connection ~ 1800 2600
+Wire Wire Line
+	2000 2700 2050 2700
+Connection ~ 2000 2700
+Wire Wire Line
+	1900 4500 1900 4650
+Wire Wire Line
+	1250 1400 2600 1400
+Wire Wire Line
+	4800 4450 4800 4950
+Connection ~ 4800 4750
+Wire Wire Line
+	2850 -1000 3300 -1000
+Wire Wire Line
+	4500 5250 4500 5300
+Wire Wire Line
+	4800 3950 4800 3900
+Wire Wire Line
+	4800 3900 5750 3900
+Wire Wire Line
+	5200 4500 5200 3900
+Connection ~ 5200 3900
+Wire Wire Line
+	5200 4900 5750 4900
+Wire Wire Line
+	4800 5850 4800 6000
+Wire Wire Line
+	2550 2600 3150 2600
+Wire Wire Line
+	2550 2700 3150 2700
+Wire Wire Line
+	2650 2700 2650 3500
+Wire Wire Line
+	2650 3500 3350 3500
+Connection ~ 2650 2700
+Wire Wire Line
+	4300 3600 4150 3600
+Wire Wire Line
+	6400 2600 6400 3500
+Wire Wire Line
+	5850 2600 6400 2600
+Wire Wire Line
+	3150 3100 2900 3100
+Wire Wire Line
+	2900 3100 2900 3700
+Wire Wire Line
+	2900 3700 3350 3700
+Wire Wire Line
 	4150 3700 4300 3700
 Wire Wire Line
 	4300 3700 4300 4000
 Wire Wire Line
-	4150 3500 6400 3500
+	6400 3500 4150 3500
 Wire Wire Line
 	4300 3300 4300 3600
@@
 Wire Wire Line
 	4800 4750 4900 4750
+$Comp
+L R R7
+U 1 1 54F9D94C
+P 2850 1400
+F 0 "R7" V 2930 1400 40  0000 C CNN
+F 1 "1k" V 2857 1401 40  0000 C CNN
+F 2 "~" V 2780 1400 30  0000 C CNN
+F 3 "~" H 2850 1400 30  0000 C CNN
+	1    2850 1400
+	0    -1   -1   0
+$EndComp
+Connection ~ 2000 1400
+Wire Wire Line
+	3100 1400 3700 1400
+Wire Wire Line
+	3700 1400 3700 1900
+Wire Wire Line
+	3700 1850 3750 1850
+$Comp
+L C C1
+U 1 1 54F9D9CA
+P 3700 2100
+F 0 "C1" H 3700 2200 40  0000 L CNN
+F 1 "100 uF" H 3706 2015 40  0000 L CNN
+F 2 "~" H 3738 1950 30  0000 C CNN
+F 3 "~" H 3700 2100 60  0000 C CNN
+	1    3700 2100
+	1    0    0    -1
+$EndComp
+Connection ~ 3700 1850
+Wire Wire Line
+	4100 2150 4100 2350
+Wire Wire Line
+	3700 2300 4100 2300
+Connection ~ 4100 2300
+Wire Wire Line
+	4500 1850 6050 1850
+Wire Wire Line
+	6050 1850 6050 2600
+Connection ~ 6050 2600
+Wire Wire Line
+	5850 3100 5850 3200
 $EndSCHEMATC
